Commit message: model23 is now the best model

File: assets/panthera-6dof.urdf (robot description, URDF)
Before this commit: robot Panthera-HT_description, 8 links, 7 joints
Joints:
- joint joint1: limit lower=-2.4 upper=2.4 effort=21 velocity=4.2 -> lower=-2.4 upper=2.4 effort=21 velocity=7.85
- joint joint2: limit lower=0.0 upper=3.2 effort=36 velocity=5 -> lower=0.0 upper=3.2 effort=36 velocity=6.28
- joint joint3: limit lower=0.0 upper=4.0 effort=36 velocity=5 -> lower=0.0 upper=4.0 effort=36 velocity=6.28
- joint joint4: limit lower=-1.6 upper=1.6 effort=21 velocity=4.2 -> lower=-1.6 upper=1.6 effort=21 velocity=7.85
- joint joint5: limit lower=-1.7 upper=1.7 effort=10 velocity=3.7 -> lower=-1.7 upper=1.7 effort=10 velocity=16.76
- joint joint6: limit lower=-2.5 upper=2.5 effort=10 velocity=3.7 -> lower=-2.5 upper=2.5 effort=10 velocity=16.76
